File: smartgarage.sch (EAGLE design)
At the start: 18 parts, among them J1 USB_MINI-B_SMT, J2 CLOSED_REED, J3 IN, J4 OUT, J5 PROG, J6 OPEN_REED, U2 ESP-12F

Commit message: V1.2 - Rotated ESP, add lock
Parts:
- removed J6: OPEN_REED, SparkFun-Connectors:CONN_023.5MM-NO_SILK
- removed R5: 10K, SparkFun-Resistors:RESISTOR0805
- removed S2: MOMENTARY-SWITCH-SPST-SMD-4.5MM, SparkFun-Switches:MOMENTARY-SWITCH-SPST-SMD-4.5MM
- added S1: MOMENTARY-SWITCH-SPST-SMD-6.2MM-TALL, SparkFun-Switches:MOMENTARY-SWITCH-SPST-SMD-6.2MM-TALL
- added U$3: LH1546, smartgarage:LH1546
- R3: value 10K -> 100
Connections:
- removed net N$3: J3.1, J4.2, U$2.S2
- new net N$7: R3.2, U$3.A
- new net N$8: J3.1, U$3.S1
- new net N$9: J4.2, U$2.S2, U$3.S2
- net 3.3V: no longer R3.2, R5.2
- net GND: now also S1.2, U$3.C; no longer J6.1, S2.2
- net GPIO12: no longer R5.1
- net GPIO13: no longer J6.2
- net N$1: now also S1.1; no longer S2.1
- net RX: now also J5.2; no longer J5.1
- net TX: now also J5.1; no longer J5.2
Other:
- moved on the sheet: J3, R3
Changed lines of the file:
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@@
 <part name="J2" library="SparkFun-Connectors" deviceset="CONN_02" device="3.5MM-NO_SILK" value="CLOSED_REED"/>
 <part name="GND4" library="SparkFun-PowerSymbols" deviceset="GND" device=""/>
-<part name="R5" library="SparkFun-Resistors" deviceset="RESISTOR" device="0805" value=" 10K"/>
 <part name="R6" library="SparkFun-Resistors" deviceset="RESISTOR" device="0805" value=" 100"/>
 <part name="GND5" library="SparkFun-PowerSymbols" deviceset="GND" device=""/>
@@
 <part name="R2" library="SparkFun-Resistors" deviceset="RESISTOR" device="0805" value=" 10K"/>
 <part name="U$2" library="smartgarage" deviceset="LH1546" device=""/>
-<part name="S2" library="SparkFun-Switches" deviceset="MOMENTARY-SWITCH-SPST" device="-SMD-4.5MM"/>
-<part name="J6" library="SparkFun-Connectors" deviceset="CONN_02" device="3.5MM-NO_SILK" value="OPEN_REED"/>
+<part name="R3" library="SparkFun-Resistors" deviceset="RESISTOR" device="0805" value=" 100"/>
 <part name="GND7" library="SparkFun-PowerSymbols" deviceset="GND" device=""/>
-<part name="R3" library="SparkFun-Resistors" deviceset="RESISTOR" device="0805" value=" 10K"/>
+<part name="U$3" library="smartgarage" deviceset="LH1546" device=""/>
+<part name="S1" library="SparkFun-Switches" deviceset="MOMENTARY-SWITCH-SPST" device="-SMD-6.2MM-TALL"/>
 </parts>
 <sheets>
@@
 <instance part="J2" gate="G$1" x="53.34" y="73.66"/>
 <instance part="GND4" gate="1" x="66.04" y="68.58"/>
-<instance part="R5" gate="G$1" x="68.58" y="76.2"/>
 <instance part="R6" gate="G$1" x="71.12" y="35.56"/>
 <instance part="GND5" gate="1" x="76.2" y="30.48" rot="R270"/>
-<instance part="J3" gate="G$1" x="124.46" y="43.18" rot="R180"/>
+<instance part="J3" gate="G$1" x="124.46" y="53.34" rot="R180"/>
 <instance part="J4" gate="G$1" x="124.46" y="30.48" rot="R180"/>
 <instance part="J5" gate="G$1" x="-33.02" y="-2.54"/>
@@
 <instance part="R2" gate="G$1" x="20.32" y="22.86" rot="R180"/>
 <instance part="U$2" gate="G$1" x="93.98" y="33.02"/>
-<instance part="S2" gate="G$1" x="35.56" y="25.4"/>
-<instance part="J6" gate="G$1" x="53.34" y="50.8"/>
-<instance part="GND7" gate="1" x="66.04" y="45.72"/>
-<instance part="R3" gate="G$1" x="68.58" y="53.34"/>
+<instance part="R3" gate="G$1" x="71.12" y="53.34"/>
+<instance part="GND7" gate="1" x="76.2" y="48.26" rot="R270"/>
+<instance part="U$3" gate="G$1" x="93.98" y="50.8"/>
+<instance part="S1" gate="G$1" x="35.56" y="25.4"/>
 </instances>
 <busses>
@@
 <junction x="43.18" y="25.4"/>
 <pinref part="U2" gate="G$1" pin="GPIO15"/>
-<pinref part="S2" gate="G$1" pin="2"/>
-</segment>
-<segment>
-<pinref part="J6" gate="G$1" pin="1"/>
-<wire x1="60.96" y1="50.8" x2="66.04" y2="50.8" width="0.1524" layer="91"/>
+<pinref part="S1" gate="G$1" pin="2"/>
+</segment>
+<segment>
+<wire x1="83.82" y1="48.26" x2="78.74" y2="48.26" width="0.1524" layer="91"/>
 <pinref part="GND7" gate="1" pin="GND"/>
-<wire x1="66.04" y1="50.8" x2="66.04" y2="48.26" width="0.1524" layer="91"/>
+<pinref part="U$3" gate="G$1" pin="C"/>
 </segment>
 </net>
@@
 </segment>
 <segment>
+<pinref part="J5" gate="G$1" pin="1"/>
+<wire x1="-27.94" y1="-5.08" x2="-17.78" y2="-5.08" width="0.1524" layer="91"/>
+<label x="-17.78" y="-5.08" size="1.016" layer="95" xref="yes"/>
+</segment>
+</net>
+<net name="RX" class="0">
+<segment>
+<pinref part="U2" gate="G$1" pin="RX"/>
+<wire x1="10.16" y1="33.02" x2="15.24" y2="33.02" width="0.1524" layer="91"/>
+<label x="15.24" y="33.02" size="1.016" layer="95" xref="yes"/>
+</segment>
+<segment>
 <pinref part="J5" gate="G$1" pin="2"/>
 <wire x1="-27.94" y1="-2.54" x2="-17.78" y2="-2.54" width="0.1524" layer="91"/>
 <label x="-17.78" y="-2.54" size="1.016" layer="95" xref="yes"/>
-</segment>
-</net>
-<net name="RX" class="0">
-<segment>
-<pinref part="U2" gate="G$1" pin="RX"/>
-<wire x1="10.16" y1="33.02" x2="15.24" y2="33.02" width="0.1524" layer="91"/>
-<label x="15.24" y="33.02" size="1.016" layer="95" xref="yes"/>
-</segment>
-<segment>
-<pinref part="J5" gate="G$1" pin="1"/>
-<wire x1="-27.94" y1="-5.08" x2="-17.78" y2="-5.08" width="0.1524" layer="91"/>
-<label x="-17.78" y="-5.08" size="1.016" layer="95" xref="yes"/>
 </segment>
 </net>
@@
 <wire x1="25.4" y1="27.94" x2="25.4" y2="25.4" width="0.1524" layer="91"/>
 <junction x="25.4" y="25.4"/>
-<pinref part="S2" gate="G$1" pin="1"/>
+<pinref part="S1" gate="G$1" pin="1"/>
 </segment>
 </net>
@@
 </segment>
 <segment>
-<pinref part="R5" gate="G$1" pin="2"/>
-<wire x1="73.66" y1="76.2" x2="78.74" y2="76.2" width="0.1524" layer="91"/>
-<label x="78.74" y="76.2" size="1.016" layer="95" xref="yes"/>
-</segment>
-<segment>
 <pinref part="J5" gate="G$1" pin="3"/>
 <wire x1="-27.94" y1="0" x2="-17.78" y2="0" width="0.1524" layer="91"/>
@@
 <wire x1="25.4" y1="22.86" x2="30.48" y2="22.86" width="0.1524" layer="91"/>
 <label x="30.48" y="22.86" size="1.016" layer="95" xref="yes"/>
-</segment>
-<segment>
-<pinref part="R3" gate="G$1" pin="2"/>
-<wire x1="73.66" y1="53.34" x2="78.74" y2="53.34" width="0.1524" layer="91"/>
-<label x="78.74" y="53.34" size="1.016" layer="95" xref="yes"/>
 </segment>
 </net>
@@
 </segment>
 <segment>
-<pinref part="R5" gate="G$1" pin="1"/>
 <pinref part="J2" gate="G$1" pin="2"/>
-<wire x1="63.5" y1="76.2" x2="61.976" y2="76.2" width="0.1524" layer="91"/>
 <wire x1="61.976" y1="76.2" x2="60.96" y2="76.2" width="0.1524" layer="91"/>
 <wire x1="61.976" y1="80.264" x2="61.976" y2="76.2" width="0.1524" layer="91"/>
-<junction x="61.976" y="76.2"/>
 <label x="61.976" y="80.264" size="1.016" layer="95" rot="R90" xref="yes"/>
 </segment>
@@
 <wire x1="114.3" y1="30.48" x2="114.3" y2="35.56" width="0.1524" layer="91"/>
 <wire x1="104.14" y1="35.56" x2="114.3" y2="35.56" width="0.1524" layer="91"/>
+<pinref part="U$2" gate="G$1" pin="S1"/>
+<wire x1="114.3" y1="35.56" x2="114.3" y2="50.8" width="0.1524" layer="91"/>
 <pinref part="J3" gate="G$1" pin="2"/>
-<wire x1="116.84" y1="40.64" x2="114.3" y2="40.64" width="0.1524" layer="91"/>
-<wire x1="114.3" y1="40.64" x2="114.3" y2="35.56" width="0.1524" layer="91"/>
+<wire x1="114.3" y1="50.8" x2="116.84" y2="50.8" width="0.1524" layer="91"/>
 <junction x="114.3" y="35.56"/>
-<pinref part="U$2" gate="G$1" pin="S1"/>
-</segment>
-</net>
-<net name="N$3" class="0">
-<segment>
+</segment>
+</net>
+<net name="N$5" class="0">
+<segment>
+<pinref part="U2" gate="G$1" pin="GPIO2"/>
+<pinref part="R2" gate="G$1" pin="2"/>
+<wire x1="10.16" y1="22.86" x2="15.24" y2="22.86" width="0.1524" layer="91"/>
+</segment>
+</net>
+<net name="GPIO13" class="0">
+<segment>
+<pinref part="U2" gate="G$1" pin="GPIO13"/>
+<wire x1="-22.86" y1="20.32" x2="-38.1" y2="20.32" width="0.1524" layer="91"/>
+<label x="-38.1" y="20.32" size="1.016" layer="95" rot="R180" xref="yes"/>
+</segment>
+<segment>
+<pinref part="R3" gate="G$1" pin="1"/>
+<wire x1="66.04" y1="53.34" x2="58.42" y2="53.34" width="0.1524" layer="91"/>
+<label x="58.42" y="53.34" size="1.016" layer="95" rot="R180" xref="yes"/>
+</segment>
+</net>
+<net name="N$7" class="0">
+<segment>
+<pinref part="R3" gate="G$1" pin="2"/>
+<wire x1="83.82" y1="53.34" x2="76.2" y2="53.34" width="0.1524" layer="91"/>
+<pinref part="U$3" gate="G$1" pin="A"/>
+</segment>
+</net>
+<net name="N$8" class="0">
+<segment>
+<wire x1="104.14" y1="53.34" x2="116.84" y2="53.34" width="0.1524" layer="91"/>
+<pinref part="U$3" gate="G$1" pin="S1"/>
 <pinref part="J3" gate="G$1" pin="1"/>
-<wire x1="116.84" y1="43.18" x2="111.76" y2="43.18" width="0.1524" layer="91"/>
+</segment>
+</net>
+<net name="N$9" class="0">
+<segment>
+<wire x1="104.14" y1="48.26" x2="111.76" y2="48.26" width="0.1524" layer="91"/>
+<pinref part="U$3" gate="G$1" pin="S2"/>
 <wire x1="104.14" y1="30.48" x2="111.76" y2="30.48" width="0.1524" layer="91"/>
 <pinref part="J4" gate="G$1" pin="2"/>
 <wire x1="111.76" y1="30.48" x2="111.76" y2="27.94" width="0.1524" layer="91"/>
 <wire x1="111.76" y1="27.94" x2="116.84" y2="27.94" width="0.1524" layer="91"/>
-<wire x1="111.76" y1="43.18" x2="111.76" y2="30.48" width="0.1524" layer="91"/>
+<pinref part="U$2" gate="G$1" pin="S2"/>
+<wire x1="111.76" y1="48.26" x2="111.76" y2="30.48" width="0.1524" layer="91"/>
 <junction x="111.76" y="30.48"/>
-<pinref part="U$2" gate="G$1" pin="S2"/>
-</segment>
-</net>
-<net name="N$5" class="0">
-<segment>
-<pinref part="U2" gate="G$1" pin="GPIO2"/>
-<pinref part="R2" gate="G$1" pin="2"/>
-<wire x1="10.16" y1="22.86" x2="15.24" y2="22.86" width="0.1524" layer="91"/>
-</segment>
-</net>
-<net name="GPIO13" class="0">
-<segment>
-<pinref part="J6" gate="G$1" pin="2"/>
-<pinref part="R3" gate="G$1" pin="1"/>
-<wire x1="60.96" y1="53.34" x2="61.976" y2="53.34" width="0.1524" layer="91"/>
-<wire x1="61.976" y1="53.34" x2="63.5" y2="53.34" width="0.1524" layer="91"/>
-<wire x1="61.976" y1="57.912" x2="61.976" y2="53.34" width="0.1524" layer="91"/>
-<junction x="61.976" y="53.34"/>
-<label x="61.976" y="57.912" size="1.016" layer="95" rot="R90" xref="yes"/>
-</segment>
-<segment>
-<pinref part="U2" gate="G$1" pin="GPIO13"/>
-<wire x1="-22.86" y1="20.32" x2="-38.1" y2="20.32" width="0.1524" layer="91"/>
-<label x="-38.1" y="20.32" size="1.016" layer="95" rot="R180" xref="yes"/>
 </segment>
 </net>
@@
 </sheet>
 </sheets>
+<errors>
+</errors>
 </schematic>
 </drawing>
